File: Blinky Flower.kicad_pcb (KiCad board)
At the start: 2 copper layers, 51.7 x 49.8 mm, 19 parts, among them J2 Conn_01x02_Socket, J3 Conn_01x01_Socket, U1 NE555P, U2 4017

Commit message: update files
Connections:
- C2 pad 2: unconnected-(C2-Pad2) -> GND
Other:
- outline, holes or cut-outs redrawn
