File: Blinky Flower.kicad_sch (KiCad schematic)
At the start: 19 parts, among them J2 Conn_01x02_Socket, J3 Conn_01x01_Socket, U1 NE555P, U2 4017

Commit message: update files
Connections:
- net GND: now also C2.2
Changed lines of the file:
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@@
+	)
+	(junction
+		(at 127 76.2)
+		(diameter 0)
+		(color 0 0 0 0)
 	)
 	(junction
@@
 		)
 		(stroke
+			(width 0)
+			(type default)
+		)
+	)
+	(wire
+		(pts
+			(xy 111.76 76.2) (xy 127 76.2)
+		)
+		(stroke
